File: CycloMod.kicad_sch (KiCad schematic)
At the start: 72 parts, among them J1 MICROMOD-2222, U1 10CL010YM164, U2 W25Q128JVS, U3 1.2V, U4 RP2350_60QFN, U5 MIC5504-2.5YMT, Y1 ABM8-272-T3

Commit message: cleaning up nets
Connections:
- net AUD_BCLK: now also U1.K15 (IO_K15_DR21N_DEVOE); no longer U1.L14 (IO_L14_DR31P)
- net AUD_IN: now also U1.L14 (IO_L14_DR31P); no longer U1.M15 (IO_M15_DR31N)
- net AUD_LRCLK: now also U1.L15 (IO_L15_VREFB5N1); no longer U1.N15 (IO_N15_RUP3)
- net AUD_OUT: now also U1.M15 (IO_M15_DR31N); no longer U1.M14 (IO_M14_RDN3)
- net SCL1: now also U1.N15 (IO_N15_RUP3); no longer U1.L15 (IO_L15_VREFB5N1)
- net SDA1: now also U1.M14 (IO_M14_RDN3); no longer U1.K15 (IO_K15_DR21N_DEVOE)
Changed lines of the file:
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@@
 	)
 	(label "SDA1"
-		(at 247.65 162.56 180)
+		(at 247.65 149.86 180)
 		(fields_autoplaced yes)
 		(effects
@@
 	)
 	(label "SCL1"
-		(at 247.65 144.78 180)
+		(at 247.65 147.32 180)
 		(fields_autoplaced yes)
 		(effects
@@
 	)
 	(label "AUD_LRCLK"
-		(at 247.65 147.32 180)
+		(at 247.65 144.78 180)
 		(fields_autoplaced yes)
 		(effects
@@
 	)
 	(label "AUD_IN"
-		(at 247.65 139.7 180)
+		(at 247.65 142.24 180)
 		(fields_autoplaced yes)
 		(effects
@@
 	)
 	(label "AUD_OUT"
-		(at 247.65 149.86 180)
+		(at 247.65 139.7 180)
 		(fields_autoplaced yes)
 		(effects
@@
 	)
 	(label "AUD_BCLK"
-		(at 247.65 142.24 180)
-		(fields_autoplaced yes)
-		(effects
+		(at 247.65 162.56 180)
+		(fields_autoplaced yes)
+		(effects

Commit message: commiting as submitted for build
Parts:
- FRAME1, J1, JP2, LOGO3, LOGO4, TP1, TP2, TP3, TP4: now fitted; now left out of the parts list
- U2: value W25Q128JVS -> W25Q128JVP
Other:
- note added: "FPGA Configuration: RP2350 is connected to JTAG This can load FPGA from on board flash using JBC player. Serial Configuration pins are connected to card edge These can be used for configuration with additional hardware on the carrier board nCONFIG is connected to !RESET This ensures it will not be driving QSPI pins when the RP2350 boots. It can be a second QSPI target after boot."
- note added: "MSEL: 000 Standard Passive Serial (Default) 010 Standard 3.3V Active Serial RP2350 is connected to JTAG Leave in passive serial to prevent FPGA from driving SPI signals when configuration is reset"

Commit message: fixed QMI SD1 pull-down, cleaned up notes
Parts:
- removed LOGO4: SPECIAL_INSTRUCTIONS-ORDERING, MicroMod-RP2040-ProcessorBoard:ORDERING_INSTRUCTIONS, symbol MicroMod-RP2040-ProcessorBoard-eagle-import:SPECIAL_INSTRUCTIONS-ORDERING
- added R15: 10k, Resistor_SMD:R_0201_0603Metric, symbol Device:R_US
- U1: value 10CL010YM164 -> 10CL016YM164
- U5: value MIC5504-2.5YMT -> XC6223-2.5V
Connections:
- net GND: now also R15.1
- net QSPI_SD1: now also R15.2
Other:
- note removed: "Board thickness: 0.8mm"
- note removed: "Dielectric thickness (layer 1 to 2): 3.93mil/0.1mm"
- note removed: "Differential Impedance: 100Ω"
- note removed: "Differential Microstrip Calculation:"
- note removed: "Er: 4.6 (JLC7628)"
- note removed: "N. Seidle"
- note removed: "Required Trace Separation: 4mil"
- note removed: "Required Trace Width: 5mil"
- note removed: "Single Ended Impedance: 50Ω"
- note removed: "Trace Thickness (1oz): 1.4mil/0.035mm"
- note removed: "https://cart.jlcpcb.com/impedanceCalculation"
- note removed: "v1.7"
- company: (none) -> Steiert Solutions
- title: (none) -> CycloMod FPGA/MCU Module

Commit message: fixed BOM and re-sync to pcb
Parts:
- U1: LCSC C1550733 -> C6063581; MPN 10CL010YM164I7G -> 10CL016YM164I7G
Changed lines of the file:
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@@
 			)
 		)
-		(property "LCSC" "C1550733"
+		(property "LCSC" "C6063581"
 			(at 276.86 139.7 0)
 			(effects
@@
 			)
 		)
-		(property "MPN" "10CL010YM164I7G"
+		(property "MPN" "10CL016YM164I7G"
 			(at 276.86 139.7 0)
 			(effects
@@
 			)
 		)
-		(property "LCSC" "C1550733"
+		(property "LCSC" "C6063581"
 			(at 278.13 189.23 0)
 			(effects
@@
 			)
 		)
-		(property "MPN" "10CL010YM164I7G"
+		(property "MPN" "10CL016YM164I7G"
 			(at 278.13 189.23 0)
 			(effects
@@
 			)
 		)
-		(property "LCSC" "C1550733"
+		(property "LCSC" "C6063581"
 			(at 277.495 88.9 0)
 			(effects
@@
 			)
 		)
-		(property "MPN" "10CL010YM164I7G"
+		(property "MPN" "10CL016YM164I7G"
 			(at 277.495 88.9 0)
 			(effects
@@
 			)
 		)
-		(property "LCSC" "C1550733"
+		(property "LCSC" "C6063581"
 			(at 277.495 242.57 0)
 			(effects
@@
 			)
 		)
-		(property "MPN" "10CL010YM164I7G"
+		(property "MPN" "10CL016YM164I7G"
 			(at 277.495 242.57 0)
 			(effects
@@
 			)
 		)
-		(property "LCSC" "C1550733"
+		(property "LCSC" "C6063581"
 			(at 278.13 30.48 0)
 			(effects
@@
 			)
 		)
-		(property "MPN" "10CL010YM164I7G"
+		(property "MPN" "10CL016YM164I7G"
 			(at 278.13 30.48 0)
 			(effects
